File: pcbs/microcontroller_board/BPC-PRP-microcontroller.kicad_pcb (KiCad board)
At the start: 2 copper layers, 40 x 100 mm, 21 parts, among them J1 Us_1, J10 Curr_probe, J11 5V, J12 Gnd, J13 I2C, J2 Us_2, J3 Us_3, J4 Line_1, J5 Line_2, J6 Motor_driver_1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

Commit message: updated arduino board, add leds
Parts:
- added LED2: ~, LED_SMD:LED_1206_3216Metric, F.Cu at (88.0, 122.9)
- added LED3: ~, LED_SMD:LED_1206_3216Metric, F.Cu at (92.0, 123.1)
- added LED4: ~, LED_SMD:LED_1206_3216Metric, F.Cu at (96.0, 122.9)
- added R4: 10k, Resistor_SMD:R_1206_3216Metric, F.Cu at (88.0, 117.0)
- added R5: 10k, Resistor_SMD:R_1206_3216Metric, F.Cu at (92.0, 117.0)
- added R6: 10k, Resistor_SMD:R_1206_3216Metric, F.Cu at (96.0, 117.0)
- LED1: value LED -> ~; footprint adafruit:1206 -> LED_SMD:LED_1206_3216Metric
- moved LED1 0.40 mm to (86.6, 51.5), turned to 0 degrees
Connections:
- A1 pad D0: unconnected-(A1-D0/RX-PadD0) -> LED_1
- A1 pad D1: unconnected-(A1-D1/TX-PadD1) -> LED_2
- A1 pad D13: unconnected-(A1-D13_SCK-PadD13) -> LED_3
- R3 pad 2: Net-(LED1-PadA) -> Net-(LED1-A)
Routing:
- net LED_3: track 0.00 -> 45.0 mm, vias 0 -> 4
- net GND: track 220.9 -> 239.7 mm
- net LED_2: track 0.00 -> 15.3 mm, vias 0 -> 1
- net LED_1: track 0.00 -> 14.4 mm, vias 0 -> 1
- net Net-(LED1-PadA): track 4.04 -> 0.00 mm
- net Net-(LED1-A): track 0.00 -> 4.04 mm
- net Net-(LED3-A): track 0.00 -> 3.20 mm
- net Net-(LED2-A): track 0.00 -> 3.08 mm
- net Net-(LED4-A): track 0.00 -> 3.00 mm
- net Net-(A1-PadA3): track 40.8 -> 38.8 mm
- net EN_2_B: track 49.9 -> 48.7 mm
- net Motor_2_B: track 63.4 -> 64.3 mm
Other:
- board text added: "uP Board Arduino v1.3.0 Adam Ligocki 28.11.2024"
- board text removed: "uP Board Arduino v1.2.0 Adam Ligocki 2024"
