File: pcbs/rpi_hat/BPC-PRP-rpi-hat.kicad_pcb (KiCad board)
At the start: 2 copper layers, 56 x 65 mm, 38 parts, among them J1 Power, J2 Power, J3 Fan_power, J4 I2C, J5 UART, J6 SPI, SW1 SW_DIP_x01, SW2 SW_DIP_x01, SW3 SW_DIP_x01, U3 DS3231M

Commit message: updated rpi ext board
Parts:
- added LED3: ~, LED_SMD:LED_1206_3216Metric, F.Cu at (149.6, 126.0)
- added LED4: ~, LED_SMD:LED_1206_3216Metric, F.Cu at (149.6, 130.0)
- added LED5: ~, LED_SMD:LED_1206_3216Metric, F.Cu at (149.6, 134.0)
- added R12: 10k, Resistor_SMD:R_1206_3216Metric, F.Cu at (154.5, 126.0)
- added R13: 10k, Resistor_SMD:R_1206_3216Metric, F.Cu at (154.5, 130.0)
- added R14: 10k, Resistor_SMD:R_1206_3216Metric, F.Cu at (154.5, 134.0)
- C4, R4, R5, R6: moved to B.Cu
- LED1, LED2: footprint adafruit:CHIPLED_1206 -> LED_SMD:LED_1206_3216Metric
- moved C4 7.83 mm to (154.5, 132.5), turned to 0 degrees
- moved R4 4.61 mm to (154.5, 130.0), turned to 180 degrees
- moved R5 4.61 mm to (154.5, 125.0), turned to 180 degrees
- moved R6 4.58 mm to (154.5, 127.5), turned to 180 degrees
- moved U3 4.28 mm to (146.0, 130.0)
- moved BT1 4.12 mm to (129.0, 130.0)
- moved LED1 0.14 mm to (121.5, 93.1), turned to 90 degrees
- moved LED2 0.11 mm to (124.0, 92.9), turned to 90 degrees
Connections:
- R7 pad 1: Net-(LED1-PadA) -> Net-(LED1-A)
- R8 pad 1: Net-(LED2-PadA) -> Net-(LED2-A)
- U1 pad 37: unconnected-(U1-GPIO_26-Pad37) -> LED_1
- U1 pad 38: unconnected-(U1-GPIO_20_(PCM_DIN)-Pad38) -> LED_2
- U1 pad 40: unconnected-(U1-GPIO_21_(PCM_DOUT)-Pad40) -> LED 3
Routing:
- net GND: track 323.0 -> 338.9 mm
- net Net-(U3-32KHZ): track 11.7 -> 2.65 mm, vias 1 -> 0
- net Net-(U3-~{RST}): track 11.2 -> 2.69 mm, vias 1 -> 0
- net LED 3: track 0.00 -> 8.26 mm
- net LED_2: track 0.00 -> 7.65 mm
- net Net-(U3-~{INT}/SQW): track 9.73 -> 2.67 mm, vias 1 -> 0
- net LED_1: track 0.00 -> 3.96 mm
- net SYS_SCL: track 43.8 -> 47.2 mm
- net SYS_SDA: track 40.7 -> 43.8 mm
- net +3V3: track 134.4 -> 137.3 mm, vias 3 -> 2
- net +BATT: track 30.0 -> 32.7 mm
- net RGB_LEDS: track 58.2 -> 60.6 mm
- net Net-(LED2-PadA): track 2.12 -> 0.00 mm
- net Net-(LED2-A): track 0.00 -> 2.12 mm
- net Net-(LED1-PadA): track 2.12 -> 0.00 mm
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Other:
- board text added: "RPi Ext. Board v1.3.0 Adam Ligocki 28.11.2024"
- board text removed: "RPi Ext. Board v1.2.0 Adam Ligocki 2024"

Commit message: add i2c pullups for rpi ext and i2c board
Parts:
- added R15: 2k2, Resistor_SMD:R_1206_3216Metric, F.Cu at (129.2, 79.3)
- added R16: 2k2, Resistor_SMD:R_1206_3216Metric, F.Cu at (126.8, 79.3)
- moved J2 3.04 mm to (123.5, 78.6)
Routing:
- net SCL: track 10.5 -> 39.5 mm
- net SDA: track 10.8 -> 34.4 mm
- net VCC: track 220.3 -> 227.3 mm
- net GND: track 338.9 -> 334.1 mm, vias 0 -> 1
- net +3V3: track 137.3 -> 141.7 mm
Other:
- board text added: "RPi Ext. Board v1.3.1 Adam Ligocki 01.12.2024"
- board text removed: "RPi Ext. Board v1.3.0 Adam Ligocki 28.11.2024"
