Commit message: T4 spec-match: real Fenrir dimensions + sensor layout + conventions
Validation pass against the actual Fenrir hardware spec (Adam,
2026-05-20) and the STL inventory in 3d-print/robot/. Changes the
URDF from "best-effort placeholder" to a sim that mirrors the real
robot in dimensions, sensor placement, polarity and topic ordering.

URDF (simulation/description/fenrir.urdf.xacro):

  * Chassis 16x14x5 cm placeholder -> 15x15x15 cm cube (matches the
    plate_bot/mid/top.STL 150x150 mm footprint, with a notional 15 cm
    height for the stacked-plate assembly + LCD/mounts on top).
  * Chassis origin shifted so its BOTTOM sits at axle level (was
    centered on the axle plane, which half-buried it).
  * Mass 0.8 kg -> 1.0 kg estimate (a 15 cm cube of robot is heavier).
  * Wheel width 20 mm -> 30 mm (per wheel.STL).
  * Wheel separation 20 cm -> 12 cm (real interwheel).
  * Wheel radius stays 33 mm (spec; STL says 34 mm, 1 mm tolerance).
  * Casters: previously one rear sphere. Now two passive sphere
    casters (front + rear, at x = ±65 mm) to mirror the real Fenrir's
    leg_front_2 skid + leg_rear_2 support + ball_2 caster -- the 15 cm
    chassis with camera weight at the front would nose-dive on a single
    rear caster.
  * LiDAR: XY-center, 20 mm above chassis top (was above a 5 cm
    placeholder chassis -> repositioned to the new ceiling).
  * Camera: front-top edge of chassis, pitched 45 deg DOWN to point
    at the ground (was looking horizontally forward).
  * Ultrasounds (3x, NEW): SRF-05-like single-ray gpu_lidar sensors at
    forward, +45 deg left, -45 deg right. All at mid-chassis height,
    sticking out 5 mm past the front face so the raycast doesn't start
    inside the chassis collision (would clamp to min_range). Side
    units sit at the front-LEFT and front-RIGHT corners.
  * Line sensors: mount moved from line_sensor_x=0.07 to caster_front_x
    (=0.065 m, same X as the front leg). The downward floor_camera
    still samples two pixels that correspond to "slightly left" and
    "slightly right" of that mount.

Sensor / topic semantics:

  * LINE SENSOR POLARITY FLIPPED: white floor -> LOW reading,
    black line -> HIGH reading. Matches the real Fenrir ADC.
  * TOPIC ORDERING CONVENTION: every multi-element /bpc_prp_robot/*
    topic is now LEFT-to-RIGHT. set_motor_speeds = [left, right],
    line_sensors = [left, right], ultrasounds = [left, center, right]
    (T4.3 stub). Fixes the previously-inverted motor command unpacking
    in motor_bridge.

Bridge updates:

  * fenrir_sim/motor_bridge.py: msg.data[0] = left wheel, msg.data[1]
    = right wheel. Doc-string lists the project-wide left-to-right
    convention.
  * fenrir_sim/line_sensor_bridge.py: brightness -> ADC mapping
    inverted; one-line change in _brightness_to_reading.

Demo controller (examples/line_follower.py):

  * Output: msg.data = [left, right] (was [right, left]).
  * err = right - left  (sign-corrected for the new polarity).
  * Added LOST state: when both sensors read below `line_threshold`,
    rotate toward the last-known line direction at a slow crawl.
    Recovers from drift / glancing corners without needing a smarter
    controller.
  * Default tuning lowered to a gentle PID: base_byte=9 (~0.09 m/s),
    kp=0.075, kd=0, no I term (verified non-aggressive by Adam
    2026-05-20).

Smoke-tested in headless and GUI modes on linux/amd64:

  * All 3 ultrasounds return inf on clear floor (no self-occlusion).
  * /bpc_prp_robot/lidar still publishing ~11.5 Hz.
  * Line-sensor polarity: ON line = [800, 810]; OFF line = [130..270]
    depending on lighting. 3-4x contrast, plenty for threshold-based
    line following.
  * Robot sits stable on both casters (no front nose-dive).
  * Line-follower drives forward, tracks straights, attempts to
    recover at the rectangular track corners via the LOST-state
    rotate.

README rewritten:

  * Status table updated to reflect the actually-shipped pieces
    (casters, ultrasounds, polarity flip, demo controller).
  * Placeholder-dimensions section replaced with a table sourced from
    the spec + STLs.
  * New "Topic-ordering convention" section so future bridge work
    (encoders, ultrasounds, RGB LEDs) follows the same left-to-right
    rule.
  * End-to-end demo section updated with the new controller logic
    (two-state machine) and current tuning values.
  * Line-sensor calibration notes describe the new polarity and
    the observed contrast.

Co-Authored-By: Claude Opus 4.7 (1M context) <noreply@anthropic.com>

File: simulation/description/fenrir.urdf.xacro (robot description, xacro)
@@ -2,33 +2,62 @@
 <!--
   Fenrir robot description for Gazebo Harmonic + ROS 2 Jazzy (Phase 4).
-  ALL DIMENSIONS BELOW ARE PLACEHOLDERS to be refined against the editable
-  SolidWorks CAD in bpc-prp-devel/hw_design/3d_model/. Values are best-effort
-  estimates based on the 3D-print STL inventory + the BPC-PRP MPC-MAP
-  reference (interwheel = 0.2 m, max body speed = 1 m/s). Cross-check before
-  using sim outputs for any quantitative claim.
+  Dimensions per spec confirmed by Adam Ligocki 2026-05-20:
+    * chassis     : 15 × 15 × 15 cm cube
+    * wheelbase   : 12 cm (interwheel)
+    * wheel       : 33 mm radius (66 mm diameter)
+    * lidar       : XY-center of the robot, on top of the chassis
+    * camera      : RPi camera, front-top of chassis, pitched 45° down
+    * ultrasounds : 3× — forward, +45° left, -45° right, mid-height
+  Wheel width, motor / caster mass, and other masses remain estimates;
+  refine from the editable SolidWorks CAD in bpc-prp-devel/hw_design/.
   Coordinate convention: +x forward, +y left, +z up. SI units (m, kg, s, rad).
+  base_link origin sits at wheel-axle level; chassis bottom sits at base_link z=0.
 -->
 <robot name="fenrir" xmlns:xacro="http://www.ros.org/wiki/xacro">
   <!-- ============================================================== -->
-  <!--  Dimensions (PLACEHOLDERS — refine from CAD)                    -->
-  <!-- ============================================================== -->
-  <xacro:property name="chassis_length" value="0.16"/>     <!-- m  -->
-  <xacro:property name="chassis_width"  value="0.14"/>     <!-- m  -->
-  <xacro:property name="chassis_height" value="0.05"/>     <!-- m  -->
-  <xacro:property name="chassis_mass"   value="0.8"/>       <!-- kg -->
-  <xacro:property name="wheel_radius"        value="0.033"/>  <!-- m  -->
-  <xacro:property name="wheel_width"         value="0.020"/>  <!-- m  -->
-  <xacro:property name="wheel_mass"          value="0.05"/>    <!-- kg -->
-  <xacro:property name="wheel_separation"    value="0.20"/>    <!-- m, interwheel, BPC-PRP reference -->
+  <!--  Dimensions                                                     -->
+  <!-- ============================================================== -->
+  <xacro:property name="chassis_length" value="0.15"/>     <!-- m  -->
+  <xacro:property name="chassis_width"  value="0.15"/>     <!-- m  -->
+  <xacro:property name="chassis_height" value="0.15"/>     <!-- m  -->
+  <xacro:property name="chassis_mass"   value="1.0"/>       <!-- kg, estimate -->
+  <xacro:property name="wheel_radius"        value="0.033"/>  <!-- m, spec; STL 34mm -->
+  <xacro:property name="wheel_width"         value="0.030"/>  <!-- m, from wheel.STL -->
+  <xacro:property name="wheel_mass"          value="0.05"/>    <!-- kg, estimate -->
+  <xacro:property name="wheel_separation"    value="0.12"/>    <!-- m, interwheel -->
   <xacro:property name="wheel_axle_x_offset" value="0.0"/>     <!-- m, axle vs base origin -->
   <xacro:property name="wheel_axle_z_offset" value="0.0"/>     <!-- m, axle height vs base origin -->
+  <!-- Real Fenrir has a FRONT skid (leg_front_2.STL) and a REAR support +
+       ball caster (leg_rear_2.STL + ball_2.STL). With a 15 cm chassis the
+       camera weight up front would tip the robot if it only had a rear
+       caster, so the sim mirrors the design with two passive casters. -->
   <xacro:property name="caster_radius" value="0.012"/>     <!-- m  -->
   <xacro:property name="caster_mass"   value="0.01"/>      <!-- kg -->
-  <xacro:property name="caster_x"      value="-0.07"/>     <!-- m, behind axle -->
-  <xacro:property name="lidar_height"     value="0.10"/>   <!-- m above base -->
-  <xacro:property name="camera_height"    value="0.13"/>   <!-- m above base -->
-  <xacro:property name="camera_x_offset"  value="0.05"/>   <!-- m, forward of base origin -->
-  <xacro:property name="line_sensor_x"    value="0.07"/>   <!-- m, forward of base origin -->
-  <xacro:property name="line_sensor_z"    value="-0.01"/>  <!-- m, below base origin (close to ground) -->
+  <xacro:property name="caster_front_x" value="0.065"/>    <!-- m, near front of 15cm chassis -->
+  <xacro:property name="caster_rear_x"  value="-0.065"/>   <!-- m, near rear of 15cm chassis -->
+  <!-- ===== Sensor placements (all relative to base_link) ===== -->
+  <!-- LiDAR: XY-center, on TOP of chassis with a small mount stub. -->
+  <xacro:property name="lidar_x"      value="0.0"/>
+  <xacro:property name="lidar_y"      value="0.0"/>
+  <xacro:property name="lidar_z"      value="${chassis_height + 0.020}"/>
+  <!-- Camera: front-top of chassis, pitched 45° down toward floor.
+       At z=chassis_height the camera sits at the top edge. Pitch = +π/4
+       rotates the camera_link's +x (gz "forward") down by 45°. -->
+  <xacro:property name="camera_x"     value="${chassis_length/2.0}"/>
+  <xacro:property name="camera_z"     value="${chassis_height}"/>
+  <xacro:property name="camera_pitch" value="${pi/4.0}"/>
+  <!-- Ultrasounds: all at mid-chassis-height. Sensors stick out 5 mm
+       past the front face so the gpu_lidar raycast does not start inside
+       the chassis collision volume (which would clamp it to min_range).
+       Left/right sit at the front-left and front-right corners. -->
+  <xacro:property name="us_x"          value="${chassis_length/2.0 + 0.005}"/>
+  <xacro:property name="us_z"          value="${chassis_height/2.0}"/>
+  <xacro:property name="us_side_y"     value="${chassis_width/2.0 - 0.010}"/>  <!-- near chassis corner -->
+  <xacro:property name="us_side_yaw"   value="${pi/4.0}"/>       <!-- 45° -->
+  <!-- Line sensors sit at the front-leg X (same x as caster_front), centered
+       laterally; the floor_camera then samples two pixel positions that
+       correspond to "slightly left" and "slightly right" of the leg. -->
+  <xacro:property name="line_sensor_x" value="${caster_front_x}"/>
+  <xacro:property name="line_sensor_z" value="-0.01"/>
   <!-- Encoder spec from MODERNIZATION_ROADMAP Appendix B. -->
   <xacro:property name="encoder_pulses_per_rev" value="576"/>
@@ -74,4 +103,6 @@
   <link name="base_link">
     <visual>
+      <!-- shift up so chassis BOTTOM = base_link z=0 (axle plane). -->
+      <origin xyz="0 0 ${chassis_height/2.0}" rpy="0 0 0"/>
       <geometry>
         <box size="${chassis_length} ${chassis_width} ${chassis_height}"/>
@@ -82,10 +113,18 @@
     </visual>
     <collision>
+      <origin xyz="0 0 ${chassis_height/2.0}" rpy="0 0 0"/>
       <geometry>
         <box size="${chassis_length} ${chassis_width} ${chassis_height}"/>
       </geometry>
     </collision>
-    <xacro:box_inertia mass="${chassis_mass}"
-                       x="${chassis_length}" y="${chassis_width}" z="${chassis_height}"/>
+    <!-- Inertial origin must sit at the chassis CoM, not at base_link. -->
+    <inertial>
+      <origin xyz="0 0 ${chassis_height/2.0}" rpy="0 0 0"/>
+      <mass value="${chassis_mass}"/>
+      <inertia
+        ixx="${chassis_mass*(chassis_width*chassis_width + chassis_height*chassis_height)/12.0}" ixy="0" ixz="0"
+        iyy="${chassis_mass*(chassis_length*chassis_length + chassis_height*chassis_height)/12.0}" iyz="0"
+        izz="${chassis_mass*(chassis_length*chassis_length + chassis_width*chassis_width)/12.0}"/>
+    </inertial>
   </link>
   <!-- ============================================================== -->
@@ -128,29 +167,29 @@
   <xacro:wheel side="right" reflect="-1"/>
   <!-- ============================================================== -->
-  <!--  Caster (rear)                                                  -->
-  <!-- ============================================================== -->
-  <link name="caster_link">
-    <visual>
-      <geometry>
-        <sphere radius="${caster_radius}"/>
-      </geometry>
-      <material name="grey"/>
-    </visual>
-    <collision>
-      <geometry>
-        <sphere radius="${caster_radius}"/>
-      </geometry>
-    </collision>
-    <xacro:sphere_inertia mass="${caster_mass}" radius="${caster_radius}"/>
-  </link>
-  <joint name="caster_joint" type="fixed">
-    <parent link="base_link"/>
-    <child  link="caster_link"/>
-    <origin xyz="${caster_x} 0 ${-(wheel_radius - caster_radius)}" rpy="0 0 0"/>
-  </joint>
-  <gazebo reference="caster_link">
-    <mu1>0.05</mu1>
-    <mu2>0.05</mu2>
-  </gazebo>
+  <!--  Casters (front + rear) — passive stabilizers                  -->
+  <!-- ============================================================== -->
+  <xacro:macro name="caster" params="suffix x">
+    <link name="caster_${suffix}_link">
+      <visual>
+        <geometry><sphere radius="${caster_radius}"/></geometry>
+        <material name="grey"/>
+      </visual>
+      <collision>
+        <geometry><sphere radius="${caster_radius}"/></geometry>
+      </collision>
+      <xacro:sphere_inertia mass="${caster_mass}" radius="${caster_radius}"/>
+    </link>
+    <joint name="caster_${suffix}_joint" type="fixed">
+      <parent link="base_link"/>
+      <child  link="caster_${suffix}_link"/>
+      <origin xyz="${x} 0 ${-(wheel_radius - caster_radius)}" rpy="0 0 0"/>
+    </joint>
+    <gazebo reference="caster_${suffix}_link">
+      <mu1>0.05</mu1>
+      <mu2>0.05</mu2>
+    </gazebo>
+  </xacro:macro>
+  <xacro:caster suffix="front" x="${caster_front_x}"/>
+  <xacro:caster suffix="rear"  x="${caster_rear_x}"/>
   <!-- ============================================================== -->
   <!--  Lidar (RPLiDAR A1 — 360° 2D scan)                             -->
@@ -175,5 +214,5 @@
     <parent link="base_link"/>
     <child  link="lidar_link"/>
-    <origin xyz="0 0 ${lidar_height}" rpy="0 0 0"/>
+    <origin xyz="${lidar_x} ${lidar_y} ${lidar_z}" rpy="0 0 0"/>
   </joint>
   <gazebo reference="lidar_link">
@@ -226,5 +265,6 @@
     <parent link="base_link"/>
     <child  link="camera_link"/>
-    <origin xyz="${camera_x_offset} 0 ${camera_height}" rpy="0 0 0"/>
+    <!-- Front-top of chassis, pitched 45° down toward the ground. -->
+    <origin xyz="${camera_x} 0 ${camera_z}" rpy="0 ${camera_pitch} 0"/>
   </joint>
   <link name="camera_optical_frame"/>
@@ -284,4 +324,63 @@
     </sensor>
   </gazebo>
+  <!-- ============================================================== -->
+  <!--  Ultrasounds (3× SRF-05-like, single-ray for now)               -->
+  <!--                                                                 -->
+  <!--  Forward, +45° left, -45° right. All at mid-chassis height.    -->
+  <!--  Gazebo Harmonic has no native sonar primitive, so we use      -->
+  <!--  single-sample gpu_lidar sensors. The T4.3 ultrasound_bridge   -->
+  <!--  (follow-up) will aggregate the three /us_* topics into a      -->
+  <!--  std_msgs/UInt8MultiArray of 3 distances in cm, matching the   -->
+  <!--  /bpc_prp_robot/ultrasounds contract in Appendix B.            -->
+  <!-- ============================================================== -->
+  <xacro:macro name="ultrasound" params="suffix x y yaw">
+    <!-- Sensor link is a 2x2x1 cm visual marker only — no collision so
+         the sensor's own model does not occlude the raycast. -->
+    <link name="us_${suffix}_link">
+      <visual>
+        <geometry><box size="0.02 0.02 0.01"/></geometry>
+        <material name="dark_grey"/>
+      </visual>
+      <xacro:box_inertia mass="0.005" x="0.02" y="0.02" z="0.01"/>
+    </link>
+    <joint name="us_${suffix}_joint" type="fixed">
+      <parent link="base_link"/>
+      <child  link="us_${suffix}_link"/>
+      <origin xyz="${x} ${y} ${us_z}" rpy="0 0 ${yaw}"/>
+    </joint>
+    <gazebo reference="us_${suffix}_link">
+      <sensor name="ultrasound_${suffix}" type="gpu_lidar">
+        <topic>us_${suffix}</topic>
+        <gz_frame_id>us_${suffix}_link</gz_frame_id>
+        <update_rate>5</update_rate>  <!-- 5 Hz per Appendix B -->
+        <lidar>
+          <scan>
+            <horizontal>
+              <samples>1</samples>
+              <min_angle>0</min_angle>
+              <max_angle>0</max_angle>
+            </horizontal>
+          </scan>
+          <range>
+            <min>0.02</min>
+            <max>2.55</max>  <!-- 255 cm max (UInt8 cap) -->
+            <resolution>0.01</resolution>
+          </range>
+          <noise>
+            <type>gaussian</type>
+            <mean>0.0</mean>
+            <stddev>0.005</stddev>
+          </noise>
+        </lidar>
+        <always_on>true</always_on>
+      </sensor>
+    </gazebo>
+  </xacro:macro>
+  <xacro:ultrasound suffix="front" x="${us_x}"
+                    y="0"                  yaw="0"/>
+  <xacro:ultrasound suffix="left"  x="${us_x}"
+                    y="${us_side_y}"       yaw="${us_side_yaw}"/>
+  <xacro:ultrasound suffix="right" x="${us_x}"
+                    y="${-us_side_y}"      yaw="${-us_side_yaw}"/>
   <!-- ============================================================== -->
   <!--  Line sensors (T4.2)                                            -->

Commit message: T4.3: ultrasound_bridge — 3× ±30° fan -> /bpc_prp_robot/ultrasounds
Models real-US echo behaviour: each sensor reports the closest
reflector inside its beam.

URDF (description/fenrir.urdf.xacro):
* Widen each of the 3 ultrasound gpu_lidar sensors from a single ray
  to a 31-sample fan spanning ±π/6 (±30° / 60° total). Range stays
  0.02 — 2.55 m (2 — 255 cm). Two new xacro:property knobs:
  us_half_fov, us_fan_samples.

Bridge config (config/ros_gz_bridge.yaml):
* GZ_TO_ROS LaserScan entries for /us_{front,left,right} → /internal/*.

New node (fenrir_sim/ultrasound_bridge.py):
* Subscribes to the 3 /internal/us_* LaserScan topics, computes
  min(finite ranges in [range_min, range_max]) per scan, clamps to
  [2, 255] cm, casts to uint8, publishes /bpc_prp_robot/ultrasounds
  UInt8MultiArray at 5 Hz per Appendix B of the modernization roadmap.
* Pre-publish behaviour: any channel without a scan yet reports 255
  (no echo) — same as a real US that has not echoed.
* Channel ordering [us_left, us_front, us_right] follows the
  encoder_bridge L-to-R convention; configurable via the
  `channel_names` launch parameter so the real-robot wiring
  (US_0/US_1/US_2 pin order) can be matched if it differs.

Wiring:
* setup.py — new ultrasound_bridge entry point.
* line/corridor/maze launch files — start the node alongside the
  other bridges; expose `channel_names` and `publish_period` as
  launch-time-overridable parameters.

Docs (simulation/README.md):
* Status row updated: ultrasounds DONE, only buttons/RGB-LEDs remain
  in T4.3.
* Topic layout table updated to drop the *(T4.3)* placeholder on
  ultrasounds and document the [left, front, right] + 2-255 cm + 255 =
  no-echo semantics.

Verified: Python AST parse + YAML parse + xacro XML well-formedness
all green. Functional sim verification requires the bpc-prp-sim:jazzy
container; not run here.

Co-Authored-By: Claude Opus 4.7 (1M context) <noreply@anthropic.com>

File: simulation/description/fenrir.urdf.xacro (robot description, xacro)
@@ -325,13 +325,20 @@
   </gazebo>
   <!-- ============================================================== -->
-  <!--  Ultrasounds (3× SRF-05-like, single-ray for now)               -->
+  <!--  Ultrasounds (3× SRF-05-like)                                   -->
   <!--                                                                 -->
   <!--  Forward, +45° left, -45° right. All at mid-chassis height.    -->
-  <!--  Gazebo Harmonic has no native sonar primitive, so we use      -->
-  <!--  single-sample gpu_lidar sensors. The T4.3 ultrasound_bridge   -->
-  <!--  (follow-up) will aggregate the three /us_* topics into a      -->
+  <!--  Gazebo Harmonic has no native sonar primitive, so we model    -->
+  <!--  each one as a narrow gpu_lidar fan spanning ±30°. The         -->
+  <!--  ultrasound_bridge node takes the MINIMUM distance across the  -->
+  <!--  fan per sensor — mirroring real-US echo behaviour: the sensor -->
+  <!--  reports the closest reflector inside its beam. Real-spec       -->
+  <!--  range 2 cm — 255 cm, per Adam 2026-05-27.                      -->
+  <!--                                                                 -->
+  <!--  The bridge aggregates the three /us_* topics into a            -->
   <!--  std_msgs/UInt8MultiArray of 3 distances in cm, matching the   -->
   <!--  /bpc_prp_robot/ultrasounds contract in Appendix B.            -->
   <!-- ============================================================== -->
+  <xacro:property name="us_half_fov"    value="${pi/6.0}"/>  <!-- ±30° -->
+  <xacro:property name="us_fan_samples" value="31"/>          <!-- ≈2°/ray -->
   <xacro:macro name="ultrasound" params="suffix x y yaw">
     <!-- Sensor link is a 2x2x1 cm visual marker only — no collision so
@@ -357,7 +364,7 @@
           <scan>
             <horizontal>
-              <samples>1</samples>
-              <min_angle>0</min_angle>
-              <max_angle>0</max_angle>
+              <samples>${us_fan_samples}</samples>
+              <min_angle>${-us_half_fov}</min_angle>
+              <max_angle>${us_half_fov}</max_angle>
             </horizontal>
           </scan>
